Commit message: Continuing with the creating of the Inverted Pendulum project from scratch. Working initial py andurdf codes

File: Pendulum_exercise/Pendulum.urdf (robot description, URDF)
Before this commit: robot myfirst, 1 links, 0 joints
Links:
- added link rail, mass 1; collision cylinder length=5 radius=0.035; visual cylinder length=.5 radius=0.035
- link Base: geometry collision box size=0.3 0.3 1.6; visual box size=0.3 0.3 1.6
Joints:
- added joint Base_rail: type fixed, parent Base, child rail, origin xyz=0 0 .78 rpy=0 -1.57075 0

Commit message: Bases and rail ready

File: Pendulum_exercise/Pendulum.urdf (robot description, URDF)
Before this commit: robot myfirst, 2 links, 1 joints
Links:
- added link Base2, mass 100; collision box size=0.3 0.3 .8; visual box size=0.3 0.3 .8
- link Base: geometry collision box size=0.3 0.3 .8; visual box size=0.3 0.3 .8
- link rail: geometry collision cylinder length=5 radius=0.035; visual cylinder length=5 radius=0.035
Joints:
- added joint Rail_Base2: type fixed, parent rail, child Base2, origin xyz=-.3 0 -2.65 rpy=0 -1.5707 0
- joint Base_rail: origin xyz=0 0 .78 rpy=0 -1.57075 0 -> xyz=2.65 0 .3 rpy=0 -1.57075 0

Commit message: pendulum setup conructed, cart moving limits defined

File: Pendulum_exercise/Pendulum.urdf (robot description, URDF)
Before this commit: robot myfirst, 3 links, 2 joints
Links:
- added link cart, mass 1; collision box size=0.15 0.15 .4; visual box size=0.15 0.15 .4
- added link pendulum, mass 100; collision box size=0.1 0.1 .8; visual box size=0.1 0.1 .8
- added link pendulumAxis, mass 100; collision box size=0.1 0.1 .1; visual box size=0.1 0.1 .1
- link Base: geometry collision box size=0.3 0.3 1.6; visual box size=0.3 0.3 1.6
- link Base2: geometry collision box size=0.3 0.3 1.6; visual box size=0.3 0.3 1.6
Joints:
- added joint cart_pendulum: type revolute, parent cart, child pendulumAxis, origin xyz=0 .15 0 rpy=0 0 0, axis 0 1 0, limit lower=1 upper=0 effort=10.0 velocity=0.5
- added joint pendulumAxis_pendulum: type fixed, parent pendulumAxis, child pendulum, origin xyz=0 0 0.45 rpy=0 0 0
- added joint rail_cart: type prismatic, parent rail, child cart, origin xyz=0 0 0 rpy=0 0 0, axis 0 0 1, limit lower=-2 upper=2 effort=0 velocity=25
- joint Base_rail: origin xyz=2.65 0 .3 rpy=0 -1.57075 0 -> xyz=2.65 0 .75 rpy=0 -1.57075 0
- joint Rail_Base2: origin xyz=-.3 0 -2.65 rpy=0 -1.5707 0 -> xyz=-.75 0 -2.65 rpy=0 -1.5707 0

Commit message: Inverted pendulum model tunned: motors provide no extra friction, to the eye the system behaves as a zero friction no controlled pendulum would behave in real world

File: Pendulum_exercise/Pendulum.urdf (robot description, URDF)
Before this commit: robot myfirst, 6 links, 5 joints
Joints:
- joint cart_pendulum: limit lower=1 upper=0 effort=10.0 velocity=0.5 -> lower=1 upper=0 effort=0 velocity=205

Commit message: First control loop achieved, no model of the system, error correction only based on error sign

File: Pendulum_exercise/Pendulum.urdf (robot description, URDF)
Before this commit: robot myfirst, 6 links, 5 joints
Joints:
- joint cart_pendulum: origin xyz=0 .15 0 rpy=0 0 0 -> xyz=0 .15 0 rpy=0 1.570796 0
