Commit message: Adding pulleys and base hight change

File: Pendulum_exercise/Pendulum_for_cart_actuation.urdf (robot description, URDF)
Before this commit: robot myfirst, 6 links, 5 joints
Links:
- added link pulley1, mass 1; collision cylinder length=.05 radius=1; visual cylinder length=.05 radius=1
- added link pulley2, mass 1; collision cylinder length=.05 radius=1; visual cylinder length=.05 radius=1
- link Base: geometry collision box size=0.3 0.3 3; visual box size=0.3 0.3 3
- link Base2: geometry collision box size=0.3 0.3 3; visual box size=0.3 0.3 3
Joints:
- added joint Base2_pulley2: type revolute, parent Base2, child pulley2, origin xyz=0 -.3 -.4 rpy=1.570796 0 0, axis 0 0 1, limit lower=-1 upper=0 effort=0 velocity=0
- added joint Base_pulley1: type revolute, parent Base, child pulley1, origin xyz=0 -.3 .4 rpy=1.570796 0 0, axis 0 0 1, limit lower=-1 upper=0 effort=0 velocity=0
- joint Base_rail: origin xyz=2.65 0 .75 rpy=0 -1.57075 0 -> xyz=2.65 0 1.4 rpy=0 -1.57075 0
- joint Rail_Base2: origin xyz=-.75 0 -2.65 rpy=0 -1.5707 0 -> xyz=-1.4 0 -2.65 rpy=0 -1.5707 0

Commit message: Fixing joint indeces and changing cart-pendulum joint to 'fixed' for explorations

File: Pendulum_exercise/Pendulum_for_cart_actuation.urdf (robot description, URDF)
Before this commit: robot myfirst, 8 links, 7 joints
Joints:
- joint cart_pendulum: axis 0 1 0 -> (none); limit lower=1 upper=0 effort=0 velocity=205 -> (none); type revolute -> fixed

Commit message: Adding PID (only P) to center cart on rail, Pendulum_cart joint is again a revolute joint

File: Pendulum_exercise/Pendulum_for_cart_actuation.urdf (robot description, URDF)
Before this commit: robot myfirst, 8 links, 7 joints
Joints:
- joint cart_pendulum: axis (none) -> 0 1 0; limit (none) -> lower=1 upper=0 effort=0 velocity=205; type fixed -> revolute
