Commit message: adding first tendon section

File: Pendulum_exercise/Pendulum_for_tendon_actuation.urdf (robot description, URDF)
Before this commit: robot myfirst, 8 links, 7 joints
Links:
- added link tendon1, mass 1; collision cylinder length=.05 radius=.1; visual cylinder length=.05 radius=.1
Joints:
- added joint pulley1_tendon1: type revolute, parent pulley1, child tendon1, origin xyz=0 1.2 0 rpy=0 0 0, axis 0 0 1, limit lower=-1 upper=0 effort=0 velocity=0
- joint Base2_pulley2: limit lower=-1 upper=0 effort=0 velocity=0 -> lower=1 upper=-1 effort=0 velocity=0
- joint Base_pulley1: limit lower=-1 upper=0 effort=0 velocity=0 -> lower=1 upper=-1 effort=0 velocity=0

Commit message: building tendon, succesfull so far

File: Pendulum_exercise/Pendulum_for_tendon_actuation.urdf (robot description, URDF)
Before this commit: robot myfirst, 9 links, 8 joints
Links:
- removed link tendon1
- added link tendon1_1, mass 1; collision cylinder length=.05 radius=.1; visual cylinder length=.05 radius=.1
- added link tendon1_2, mass 1; collision cylinder length=.05 radius=.1; visual cylinder length=.05 radius=.1
- added link tendon1_3, mass 1; collision cylinder length=.05 radius=.1; visual cylinder length=.05 radius=.1
Joints:
- removed joint pulley1_tendon1
- added joint pulley1_tendon1_1: type revolute, parent pulley1, child tendon1_1, origin xyz=.1 1.1 0 rpy=0 0 0, axis 0 0 1, limit lower=1 upper=-1 effort=0 velocity=0
- added joint tendon1_1_tendon1_2: type revolute, parent tendon1_1, child tendon1_2, origin xyz=.2 .4 0 rpy=0 0 0, axis 0 0 1, limit lower=-1 upper=0 effort=0 velocity=0
- added joint tendon1_2_tendon1_3: type revolute, parent tendon1_2, child tendon1_3, origin xyz=.2 .4 0 rpy=0 0 0, axis 0 0 1, limit lower=-1 upper=0 effort=0 velocity=0

Commit message: A slack tendon can be seen

File: Pendulum_exercise/Pendulum_for_tendon_actuation.urdf (robot description, URDF)
Before this commit: robot myfirst, 11 links, 10 joints
Links:
- added link tendon1_4, mass 1; collision cylinder length=.05 radius=.1; visual cylinder length=.05 radius=.1
- added link tendon1_5, mass 1; collision cylinder length=.05 radius=.1; visual cylinder length=.05 radius=.1
- added link tendon1_6, mass 1; collision cylinder length=.05 radius=.1; visual cylinder length=.05 radius=.1
- added link tendon1_7, mass 1; collision cylinder length=.05 radius=.1; visual cylinder length=.05 radius=.1
Joints:
- added joint tendon1_3_tendon1_4: type revolute, parent tendon1_3, child tendon1_4, origin xyz=.2 .4 0 rpy=0 0 0, axis 0 0 1, limit lower=0 upper=-1 effort=0 velocity=0
- added joint tendon1_4_tendon1_5: type revolute, parent tendon1_4, child tendon1_5, origin xyz=.2 .4 0 rpy=0 0 0, axis 0 0 1, limit lower=0 upper=-1 effort=0 velocity=0
- added joint tendon1_5_tendon1_6: type revolute, parent tendon1_5, child tendon1_6, origin xyz=.2 .4 0 rpy=0 0 0, axis 0 0 1, limit lower=0 upper=-1 effort=0 velocity=0
- added joint tendon1_6_tendon1_7: type revolute, parent tendon1_6, child tendon1_7, origin xyz=.2 .4 0 rpy=0 0 0, axis 0 0 1, limit lower=0 upper=-1 effort=0 velocity=0
- joint tendon1_1_tendon1_2: limit lower=-1 upper=0 effort=0 velocity=0 -> lower=0 upper=-1 effort=0 velocity=0
- joint tendon1_2_tendon1_3: limit lower=-1 upper=0 effort=0 velocity=0 -> lower=0 upper=-1 effort=0 velocity=0

Commit message: tendon initial state is now horizontal, in line with rail and cart

File: Pendulum_exercise/Pendulum_for_tendon_actuation.urdf (robot description, URDF)
Before this commit: robot myfirst, 15 links, 14 joints
Joints:
- joint Base2_pulley2: origin xyz=0 -.3 -.4 rpy=1.570796 0 0 -> xyz=0 -.3 -1.4 rpy=1.570796 0 0
- joint Base_pulley1: origin xyz=0 -.3 .4 rpy=1.570796 0 0 -> xyz=0 -.3 1.4 rpy=1.570796 0 0
- joint pulley1_tendon1_1: origin xyz=.1 1.1 0 rpy=0 0 0 -> xyz=1 0 0 rpy=0 0 0
- joint tendon1_1_tendon1_2: origin xyz=.2 .4 0 rpy=0 0 0 -> xyz=.3 0 0 rpy=0 0 0
- joint tendon1_2_tendon1_3: origin xyz=.2 .4 0 rpy=0 0 0 -> xyz=.3 0 0 rpy=0 0 0
- joint tendon1_3_tendon1_4: origin xyz=.2 .4 0 rpy=0 0 0 -> xyz=.3 0 0 rpy=0 0 0
- joint tendon1_4_tendon1_5: origin xyz=.2 .4 0 rpy=0 0 0 -> xyz=.3 0 0 rpy=0 0 0
- joint tendon1_5_tendon1_6: origin xyz=.2 .4 0 rpy=0 0 0 -> xyz=.3 0 0 rpy=0 0 0
- joint tendon1_6_tendon1_7: origin xyz=.2 .4 0 rpy=0 0 0 -> xyz=.3 0 0 rpy=0 0 0

Commit message: finding a way to connect a bodies 'creation of a loop connection, problematic

File: Pendulum_exercise/Pendulum_for_tendon_actuation.urdf (robot description, URDF)
Before this commit: robot myfirst, 15 links, 14 joints
Joints:
- added joint cart_tendon1_7: type revolute, parent cart, child tendon1_7, origin xyz=0 -.3 .15 rpy=-1.570796 0 0, axis 0 0 1, limit lower=0 upper=-1 effort=0 velocity=0
- joint Base2_pulley2: origin xyz=0 -.3 -1.4 rpy=1.570796 0 0 -> xyz=0 -.3 -1.5 rpy=1.570796 0 0
- joint Base_pulley1: origin xyz=0 -.3 1.4 rpy=1.570796 0 0 -> xyz=0 -.3 1.5 rpy=1.570796 0 0
- joint Base_rail: origin xyz=2.65 0 1.4 rpy=0 -1.57075 0 -> xyz=2.65 0 1.5 rpy=0 -1.570796 0
- joint Rail_Base2: origin xyz=-1.4 0 -2.65 rpy=0 -1.5707 0 -> xyz=-1.5 0 -2.65 rpy=0 -1.570796 0
