Commit message: Cyclic body chain exploration 2

File: Pendulum_exercise/Cyclic_body_chain.urdf (robot description, URDF)
Before this commit: robot myfirst, 15 links, 15 joints
Links:
- removed link Base2
- removed link cart
- removed link pendulum
- removed link pendulumAxis
- removed link pulley1
- removed link pulley2
- removed link rail
- removed link tendon1_1
- removed link tendon1_2
- removed link tendon1_3
- removed link tendon1_4
- removed link tendon1_5
- removed link tendon1_6
- removed link tendon1_7
- added link arm1, mass 100; collision box size=0.1 0.1 1; visual box size=0.1 0.1 1
- added link axis1, mass 100; collision box size=0.1 0.1 0.1; visual box size=0.1 0.1 0.1
- added link base2, mass 100; collision box size=0.3 0.3 3; visual box size=0.3 0.3 1
- added link base3, mass 100; collision box size=0.3 0.3 3; visual box size=0.3 0.3 1
- link Base: geometry collision box size=0.3 0.3 3; visual box size=0.3 0.3 1
Joints:
- removed joint Base2_pulley2
- removed joint Base_pulley1
- removed joint Base_rail
- removed joint Rail_Base2
- removed joint cart_pendulum
- removed joint cart_tendon1_7
- removed joint pendulumAxis_pendulum
- removed joint pulley1_tendon1_1
- removed joint rail_cart
- removed joint tendon1_1_tendon1_2
- removed joint tendon1_2_tendon1_3
- removed joint tendon1_3_tendon1_4
- removed joint tendon1_4_tendon1_5
- removed joint tendon1_5_tendon1_6
- removed joint tendon1_6_tendon1_7
- added joint Base_axis1: type fixed, parent Base, child axis1, origin xyz=.1 .2 .45 rpy=0 0 0
- added joint axis1_arm1: type fixed, parent axis1, child arm1, origin xyz=0 0 .55 rpy=0 0 0
- added joint base1_base2: type fixed, parent Base, child base2, origin xyz=.65 0 -.35 rpy=0 1.57075 0
- added joint base2_base3: type fixed, parent base2, child base3, origin xyz=-.35 0 .65 rpy=0 1.57075 0

Commit message: Cyclic body chain exploration 3

File: Pendulum_exercise/Cyclic_body_chain.urdf (robot description, URDF)
Before this commit: robot myfirst, 5 links, 4 joints
Links:
- added link arm2, mass 100; collision box size=0.1 0.1 1; visual box size=0.1 0.1 1
- added link arm3, mass 100; collision box size=0.1 0.1 1; visual box size=0.1 0.1 1
- added link axis2, mass 100; collision box size=0.1 0.1 0.1; visual box size=0.1 0.1 0.1
- added link axis3, mass 100; collision box size=0.1 0.1 0.1; visual box size=0.1 0.1 0.1
Joints:
- added joint arm1_axis2: type fixed, parent arm1, child axis2, origin xyz=0 .1 .45 rpy=0 0 0
- added joint arm2_axis3: type fixed, parent arm2, child axis3, origin xyz=0 0 .55 rpy=0 0 0
- added joint axis2_arm2: type fixed, parent axis2, child arm2, origin xyz=.55 0 0 rpy=0 1.57075 0
- added joint axis3_arm3: type fixed, parent axis3, child arm3, origin xyz=0.45 -0.1 0 rpy=0 1.57075 0

Commit message: Adding physical constraint to achieve cyclic body chain

File: Pendulum_exercise/Cyclic_body_chain.urdf (robot description, URDF)
Before this commit: robot myfirst, 9 links, 8 joints
Links:
- added link axis4, mass 100; collision box size=0.1 0.1 0.1; visual box size=0.1 0.1 0.1
- added link base4, mass 100; collision box size=0.1 0.1 .3; visual box size=0.1 0.1 .3
- added link base5, mass 100; collision box size=0.1 0.1 .3; visual box size=0.1 0.1 .3
- added link base6, mass 100; collision box size=0.1 0.1 .3; visual box size=0.1 0.1 .3
- link Base: geometry collision box size=0.3 0.3 1; visual box size=0.3 0.3 1
- link base2: geometry collision box size=0.3 0.3 1; visual box size=0.3 0.3 1
- link base3: geometry collision box size=0.3 0.3 .9; visual box size=0.3 0.3 .9
Joints:
- added joint arm3_axis4: type fixed, parent arm3, child axis4, origin xyz=0 0 .55 rpy=0 0 0
- added joint base3_base4: type fixed, parent base3, child base4, origin xyz=.21 .09 -.45 rpy=0 0 0
- added joint base3_base5: type fixed, parent base3, child base5, origin xyz=-0.01 .09 -.45 rpy=0 0 0
- added joint base3_base6: type fixed, parent base3, child base6, origin xyz=.1 .1 -.61 rpy=0 1.57075 0
- joint base2_base3: origin xyz=-.35 0 .65 rpy=0 1.57075 0 -> xyz=-.30 0 .65 rpy=0 1.57075 0

Commit message: cylic body chain body achieved, not by declaration but by physical constraints

File: Pendulum_exercise/Cyclic_body_chain.urdf (robot description, URDF)
Before this commit: robot myfirst, 13 links, 12 joints
Links:
- added link axis5, mass 100; collision box size=0.1 0.1 0.1; visual box size=0.1 0.1 0.1
- link base3: geometry collision box size=0.3 0.3 .9; visual box size=0.3 0.3 .89
Joints:
- added joint axis4_axis5: type revolute, parent axis4, child axis5, origin xyz=0 -.1 0 rpy=0 0 0, axis 0 1 0, limit lower=1 upper=0 effort=0 velocity=205
- joint Base_axis1: axis (none) -> 0 1 0; limit (none) -> lower=1 upper=0 effort=0 velocity=205; type fixed -> revolute
- joint arm1_axis2: axis (none) -> 0 1 0; limit (none) -> lower=1 upper=0 effort=0 velocity=205; type fixed -> revolute
- joint arm2_axis3: axis (none) -> 0 1 0; limit (none) -> lower=1 upper=0 effort=0 velocity=205; type fixed -> revolute
- joint base2_base3: origin xyz=-.30 0 .65 rpy=0 1.57075 0 -> xyz=-.295 0 .65 rpy=0 1.57075 0
- joint base3_base6: origin xyz=.1 .1 -.61 rpy=0 1.57075 0 -> xyz=.1 .09 -.61 rpy=0 1.57075 0

Commit message: Freechain (not trapped)

File: Pendulum_exercise/Cyclic_body_chain.urdf (robot description, URDF)
Before this commit: robot myfirst, 14 links, 13 joints
Links:
- link base2: geometry collision box size=0.3 0.3 2; visual box size=0.3 0.3 2
Joints:
- joint base1_base2: origin xyz=.65 0 -.35 rpy=0 1.57075 0 -> xyz=1.15 0 -.35 rpy=0 1.57075 0
- joint base2_base3: origin xyz=-.295 0 .65 rpy=0 1.57075 0 -> xyz=-.295 0 1.15 rpy=0 1.57075 0

Commit message: chain created without self colisions

File: Pendulum_exercise/Cyclic_body_chain.urdf (robot description, URDF)
Before this commit: robot myfirst, 14 links, 13 joints
Links:
- link arm2: geometry collision box size=0.1 0.1 2; visual box size=0.1 0.1 2
Joints:
- joint arm2_axis3: origin xyz=0 0 .55 rpy=0 0 0 -> xyz=0 0 1.05 rpy=0 0 0
- joint axis2_arm2: origin xyz=.55 0 0 rpy=0 1.57075 0 -> xyz=1.05 0 0 rpy=0 1.57075 0

Commit message: Before going to pulley instead of arms

File: Pendulum_exercise/Cyclic_body_chain.urdf (robot description, URDF)
Before this commit: robot myfirst, 14 links, 13 joints
Joints:
- joint arm1_axis2: origin xyz=0 .1 .45 rpy=0 0 0 -> xyz=0 0 .65 rpy=0 0 0
- joint axis3_arm3: origin xyz=0.45 -0.1 0 rpy=0 1.57075 0 -> xyz=0.65 0 0 rpy=0 1.57075 0

Commit message: Tendon built up to cart, no rails yat

File: Pendulum_exercise/Cyclic_body_chain.urdf (robot description, URDF)
Before this commit: robot myfirst, 14 links, 13 joints
Links:
- removed link arm1
- removed link arm2
- removed link arm3
- removed link axis1
- removed link axis2
- removed link axis3
- removed link axis4
- removed link axis5
- added link cart, mass 100; collision box size=0.1 0.6 .1; visual box size=0.3 0.6 .1
- added link pulley1, mass 100; collision cylinder length=.1 radius=.5; visual cylinder length=.1 radius=.5
- added link tendon1_1, mass 10; collision cylinder length=.1 radius=.05; visual cylinder length=.1 radius=.05
- added link tendon1_2, mass 10; collision cylinder length=.1 radius=.05; visual cylinder length=.1 radius=.05
- added link tendon1_3, mass 10; collision cylinder length=.1 radius=.05; visual cylinder length=.1 radius=.05
- added link tendon1_4, mass 10; collision cylinder length=.1 radius=.05; visual cylinder length=.1 radius=.05
- added link tendon1_5, mass 10; collision cylinder length=.1 radius=.05; visual cylinder length=.1 radius=.05
- added link tendon1_6, mass 10; collision cylinder length=.1 radius=.05; visual cylinder length=.1 radius=.05
- added link tendon1_7, mass 10; collision cylinder length=.1 radius=.05; visual cylinder length=.1 radius=.05
- added link tendon1_8, mass 10; collision cylinder length=.1 radius=.05; visual cylinder length=.1 radius=.05
- added link tendon1_9, mass 10; collision cylinder length=.1 radius=.05; visual cylinder length=.1 radius=.05
- link base2: geometry collision box size=0.3 0.3 4; visual box size=0.3 0.3 4
Joints:
- removed joint Base_axis1
- removed joint arm1_axis2
- removed joint arm2_axis3
- removed joint arm3_axis4
- removed joint axis1_arm1
- removed joint axis2_arm2
- removed joint axis3_arm3
- removed joint axis4_axis5
- added joint Base_pulley1: type revolute, parent Base, child pulley1, origin xyz=.1 .21 .45 rpy=1.57075 0 0, axis 0 0 1, limit lower=1 upper=0 effort=0 velocity=205
- added joint pulley1_tendon1_1: type revolute, parent pulley1, child tendon1_1, origin xyz=0 .55 0 rpy=0 0 0, axis 0 0 1, limit lower=1 upper=0 effort=0 velocity=205
- added joint tendon1_1_tendon1_2: type revolute, parent tendon1_1, child tendon1_2, origin xyz=.2 0 0 rpy=0 0 0, axis 0 0 1, limit lower=1 upper=0 effort=0 velocity=205
- added joint tendon1_2_tendon1_3: type revolute, parent tendon1_2, child tendon1_3, origin xyz=.2 0 0 rpy=0 0 0, axis 0 0 1, limit lower=1 upper=0 effort=0 velocity=205
- added joint tendon1_3_tendon1_4: type revolute, parent tendon1_3, child tendon1_4, origin xyz=.2 0 0 rpy=0 0 0, axis 0 0 1, limit lower=1 upper=0 effort=0 velocity=205
- added joint tendon1_4_tendon1_5: type revolute, parent tendon1_4, child tendon1_5, origin xyz=.2 0 0 rpy=0 0 0, axis 0 0 1, limit lower=1 upper=0 effort=0 velocity=205
- added joint tendon1_5_tendon1_6: type revolute, parent tendon1_5, child tendon1_6, origin xyz=.2 0 0 rpy=0 0 0, axis 0 0 1, limit lower=1 upper=0 effort=0 velocity=205
- added joint tendon1_6_tendon1_7: type revolute, parent tendon1_6, child tendon1_7, origin xyz=.2 0 0 rpy=0 0 0, axis 0 0 1, limit lower=1 upper=0 effort=0 velocity=205
- added joint tendon1_7_tendon1_8: type revolute, parent tendon1_7, child tendon1_8, origin xyz=.2 0 0 rpy=0 0 0, axis 0 0 1, limit lower=1 upper=0 effort=0 velocity=205
- added joint tendon1_8_tendon1_9: type revolute, parent tendon1_8, child tendon1_9, origin xyz=.2 0 0 rpy=0 0 0, axis 0 0 1, limit lower=1 upper=0 effort=0 velocity=205
- added joint tendon1_9_cart: type fixed, parent tendon1_9, child cart, origin xyz=.45 0 0 rpy=-1.57075 0 0, axis 0 0 1, limit lower=1 upper=0 effort=0 velocity=205
- joint base1_base2: origin xyz=1.15 0 -.35 rpy=0 1.57075 0 -> xyz=2.15 0 -.35 rpy=0 1.57075 0
- joint base2_base3: origin xyz=-.295 0 1.15 rpy=0 1.57075 0 -> xyz=-.295 0 2.15 rpy=0 1.57075 0

Commit message: finished chain, but sometimes it 'breakes'(collisions are not respected)

File: Pendulum_exercise/Cyclic_body_chain.urdf (robot description, URDF)
Before this commit: robot myfirst, 17 links, 16 joints
Links:
- added link axis2, mass 10; collision cylinder length=.1 radius=.047; visual cylinder length=.1 radius=.047
- added link cube, mass 100; collision box size=0.1 0.1 0.1; visual box size=0.1 0.1 0.1
- added link pulley2, mass 10; collision cylinder length=.1 radius=.5; visual cylinder length=.1 radius=.5
- added link tendon2_1, mass 10; collision cylinder length=.1 radius=.05; visual cylinder length=.1 radius=.05
- added link tendon2_2, mass 10; collision cylinder length=.1 radius=.05; visual cylinder length=.1 radius=.05
- added link tendon2_3, mass 10; collision cylinder length=.1 radius=.05; visual cylinder length=.1 radius=.05
- added link tendon2_4, mass 10; collision cylinder length=.1 radius=.05; visual cylinder length=.1 radius=.05
- added link tendon2_5, mass 10; collision cylinder length=.1 radius=.05; visual cylinder length=.1 radius=.05
- added link tendon2_6, mass 10; collision cylinder length=.1 radius=.05; visual cylinder length=.1 radius=.05
- added link tendon2_7, mass 10; collision cylinder length=.1 radius=.05; visual cylinder length=.1 radius=.05
- added link tendon2_8, mass 10; collision cylinder length=.1 radius=.05; visual cylinder length=.1 radius=.05
- added link tendon2_9, mass 10; collision cylinder length=.1 radius=.05; visual cylinder length=.1 radius=.05
Joints:
- added joint axis2_cube: type revolute, parent axis2, child cube, origin xyz=0 0 .1 rpy=0 0 0, axis 0 0 1, limit lower=1 upper=0 effort=0 velocity=205
- added joint cart_tendon2_1: type revolute, parent cart, child tendon2_1, origin xyz=.45 0 0 rpy=1.57075 0 0, axis 0 0 1, limit lower=1 upper=0 effort=0 velocity=205
- added joint pulley2_axis2: type fixed, parent pulley2, child axis2, origin xyz=0 0 .05 rpy=0 0 0
- added joint tendon2_1_tendon2_2: type revolute, parent tendon2_1, child tendon2_2, origin xyz=.2 0 0 rpy=0 0 0, axis 0 0 1, limit lower=1 upper=0 effort=0 velocity=205
- added joint tendon2_2_tendon2_3: type revolute, parent tendon2_2, child tendon2_3, origin xyz=.2 0 0 rpy=0 0 0, axis 0 0 1, limit lower=1 upper=0 effort=0 velocity=205
- added joint tendon2_3_tendon2_4: type revolute, parent tendon2_3, child tendon2_4, origin xyz=.2 0 0 rpy=0 0 0, axis 0 0 1, limit lower=1 upper=0 effort=0 velocity=205
- added joint tendon2_4_tendon2_5: type revolute, parent tendon2_4, child tendon2_5, origin xyz=.2 0 0 rpy=0 0 0, axis 0 0 1, limit lower=1 upper=0 effort=0 velocity=205
- added joint tendon2_5_tendon2_6: type revolute, parent tendon2_5, child tendon2_6, origin xyz=.2 0 0 rpy=0 0 0, axis 0 0 1, limit lower=1 upper=0 effort=0 velocity=205
- added joint tendon2_6_tendon2_7: type revolute, parent tendon2_6, child tendon2_7, origin xyz=.2 0 0 rpy=0 0 0, axis 0 0 1, limit lower=1 upper=0 effort=0 velocity=205
- added joint tendon2_7_tendon2_8: type revolute, parent tendon2_7, child tendon2_8, origin xyz=.2 0 0 rpy=0 0 0, axis 0 0 1, limit lower=1 upper=0 effort=0 velocity=205
- added joint tendon2_8_tendon2_9: type revolute, parent tendon2_8, child tendon2_9, origin xyz=.2 0 0 rpy=0 0 0, axis 0 0 1, limit lower=1 upper=0 effort=0 velocity=205
- added joint tendon2_9_pulley2: type fixed, parent tendon2_9, child pulley2, origin xyz=0 -.55 0 rpy=0 0 0

Commit message: reduce the times the body chain breaks, an option might be to reduce the joint velocity

File: Pendulum_exercise/Cyclic_body_chain.urdf (robot description, URDF)
Before this commit: robot myfirst, 29 links, 28 joints
Joints:
- joint Base_pulley1: limit lower=1 upper=0 effort=0 velocity=205 -> lower=1 upper=0 effort=0 velocity=50
- joint axis2_cube: limit lower=1 upper=0 effort=0 velocity=205 -> lower=1 upper=0 effort=0 velocity=50
- joint cart_tendon2_1: limit lower=1 upper=0 effort=0 velocity=205 -> lower=1 upper=0 effort=0 velocity=50
- joint pulley1_tendon1_1: limit lower=1 upper=0 effort=0 velocity=205 -> lower=1 upper=0 effort=0 velocity=50
- joint tendon1_1_tendon1_2: limit lower=1 upper=0 effort=0 velocity=205 -> lower=1 upper=0 effort=0 velocity=50
- joint tendon1_2_tendon1_3: limit lower=1 upper=0 effort=0 velocity=205 -> lower=1 upper=0 effort=0 velocity=50
- joint tendon1_3_tendon1_4: limit lower=1 upper=0 effort=0 velocity=205 -> lower=1 upper=0 effort=0 velocity=50
- joint tendon1_4_tendon1_5: limit lower=1 upper=0 effort=0 velocity=205 -> lower=1 upper=0 effort=0 velocity=50
- joint tendon1_5_tendon1_6: limit lower=1 upper=0 effort=0 velocity=205 -> lower=1 upper=0 effort=0 velocity=50
- joint tendon1_6_tendon1_7: limit lower=1 upper=0 effort=0 velocity=205 -> lower=1 upper=0 effort=0 velocity=50
- joint tendon1_7_tendon1_8: limit lower=1 upper=0 effort=0 velocity=205 -> lower=1 upper=0 effort=0 velocity=50
- joint tendon1_8_tendon1_9: limit lower=1 upper=0 effort=0 velocity=205 -> lower=1 upper=0 effort=0 velocity=50
- joint tendon1_9_cart: limit lower=1 upper=0 effort=0 velocity=205 -> lower=1 upper=0 effort=0 velocity=50
- joint tendon2_1_tendon2_2: limit lower=1 upper=0 effort=0 velocity=205 -> lower=1 upper=0 effort=0 velocity=50
- joint tendon2_2_tendon2_3: limit lower=1 upper=0 effort=0 velocity=205 -> lower=1 upper=0 effort=0 velocity=50
- joint tendon2_3_tendon2_4: limit lower=1 upper=0 effort=0 velocity=205 -> lower=1 upper=0 effort=0 velocity=50
- joint tendon2_4_tendon2_5: limit lower=1 upper=0 effort=0 velocity=205 -> lower=1 upper=0 effort=0 velocity=50
- joint tendon2_5_tendon2_6: limit lower=1 upper=0 effort=0 velocity=205 -> lower=1 upper=0 effort=0 velocity=50
- joint tendon2_6_tendon2_7: limit lower=1 upper=0 effort=0 velocity=205 -> lower=1 upper=0 effort=0 velocity=50
- joint tendon2_7_tendon2_8: limit lower=1 upper=0 effort=0 velocity=205 -> lower=1 upper=0 effort=0 velocity=50
- joint tendon2_8_tendon2_9: limit lower=1 upper=0 effort=0 velocity=205 -> lower=1 upper=0 effort=0 velocity=50

Commit message: Adding variables to xml to change more easily joint velocity

File: Pendulum_exercise/Cyclic_body_chain.urdf (robot description, URDF)
Before this commit: robot myfirst, 29 links, 28 joints
Joints:
- joint axis2_cube: limit lower=1 upper=0 effort=0 velocity=50 -> lower=1 upper=0 effort=0 velocity=vel

Commit message: Longer tendon, still seing colission problems

File: Pendulum_exercise/Cyclic_body_chain.urdf (robot description, URDF)
Before this commit: robot myfirst, 29 links, 28 joints
Links:
- added link tendon2_10, mass 10; collision cylinder length=.1 radius=.05; visual cylinder length=.1 radius=.05
- added link tendon2_11, mass 10; collision cylinder length=.1 radius=.05; visual cylinder length=.1 radius=.05
- added link tendon2_12, mass 10; collision cylinder length=.1 radius=.05; visual cylinder length=.1 radius=.05
- added link tendon2_13, mass 10; collision cylinder length=.1 radius=.05; visual cylinder length=.1 radius=.05
- added link tendon2_14, mass 10; collision cylinder length=.1 radius=.05; visual cylinder length=.1 radius=.05
- added link tendon2_15, mass 10; collision cylinder length=.1 radius=.05; visual cylinder length=.1 radius=.05
- added link tendon2_16, mass 10; collision cylinder length=.1 radius=.05; visual cylinder length=.1 radius=.05
Joints:
- removed joint tendon2_9_pulley2
- added joint tendon2_10_tendon2_11: type revolute, parent tendon2_10, child tendon2_11, origin xyz=.2 0 0 rpy=0 0 -.364, axis 0 0 1, limit lower=1 upper=0 effort=0 velocity=50
- added joint tendon2_11_tendon2_12: type revolute, parent tendon2_11, child tendon2_12, origin xyz=.2 0 0 rpy=0 0 -.364, axis 0 0 1, limit lower=1 upper=0 effort=0 velocity=50
- added joint tendon2_12_tendon2_13: type revolute, parent tendon2_12, child tendon2_13, origin xyz=.2 0 0 rpy=0 0 -.364, axis 0 0 1, limit lower=1 upper=0 effort=0 velocity=50
- added joint tendon2_13_tendon2_14: type revolute, parent tendon2_13, child tendon2_14, origin xyz=.2 0 0 rpy=0 0 -.364, axis 0 0 1, limit lower=1 upper=0 effort=0 velocity=50
- added joint tendon2_14_tendon2_15: type revolute, parent tendon2_14, child tendon2_15, origin xyz=.2 0 0 rpy=0 0 -.364, axis 0 0 1, limit lower=1 upper=0 effort=0 velocity=50
- added joint tendon2_15_tendon2_16: type revolute, parent tendon2_15, child tendon2_16, origin xyz=.2 0 0 rpy=0 0 -.364, axis 0 0 1, limit lower=1 upper=0 effort=0 velocity=50
- added joint tendon2_16_pulley2: type fixed, parent tendon2_16, child pulley2, origin xyz=0 -.55 0 rpy=0 0 0
- added joint tendon2_9_tendon2_10: type revolute, parent tendon2_9, child tendon2_10, origin xyz=.2 0 0 rpy=0 0 -.364, axis 0 0 1, limit lower=1 upper=0 effort=0 velocity=50
- joint tendon2_8_tendon2_9: origin xyz=.2 0 0 rpy=0 0 0 -> xyz=.2 0 0 rpy=0 0 -.364

Commit message: Tidying up files

File: Pendulum_exercise/Cyclic_body_chain.urdf (robot description, URDF)
Before this commit: robot myfirst, 36 links, 35 joints
Links:
- removed link axis2
- removed link cube
- removed link pulley2
- removed link tendon1_6
- removed link tendon1_7
- removed link tendon1_8
- removed link tendon1_9
Joints:
- removed joint axis2_cube
- removed joint pulley2_axis2
- removed joint tendon1_5_tendon1_6
- removed joint tendon1_6_tendon1_7
- removed joint tendon1_7_tendon1_8
- removed joint tendon1_8_tendon1_9
- removed joint tendon1_9_cart
- removed joint tendon2_16_pulley2
- added joint tendon1_5_cart: type fixed, parent tendon1_5, child cart, origin xyz=.45 0 0 rpy=-1.57075 0 0, axis 0 0 1, limit lower=1 upper=0 effort=0 velocity=50
- joint tendon1_1_tendon1_2: origin xyz=.2 0 0 rpy=0 0 0 -> xyz=.4 0 0 rpy=0 0 0
- joint tendon1_2_tendon1_3: origin xyz=.2 0 0 rpy=0 0 0 -> xyz=.4 0 0 rpy=0 0 0
- joint tendon1_3_tendon1_4: origin xyz=.2 0 0 rpy=0 0 0 -> xyz=.4 0 0 rpy=0 0 0
- joint tendon1_4_tendon1_5: origin xyz=.2 0 0 rpy=0 0 0 -> xyz=.4 0 0 rpy=0 0 0
