Commit message: Adding explanation, and organizing files

File: Pendulum_exercise/Inverted_pendulum_tendon_actuation/Cyclic_body_chain.urdf (robot description, URDF)
Before this commit: robot myfirst, 29 links, 28 joints
Links:
- added link axis2, mass 10; collision cylinder length=.1 radius=.047; visual cylinder length=.1 radius=.047
- added link cube, mass 100; collision box size=0.1 0.1 0.1; visual box size=0.1 0.1 0.1
- added link pulley2, mass 10; collision cylinder length=.1 radius=.5; visual cylinder length=.1 radius=.5
Joints:
- added joint axis2_cube: type revolute, parent axis2, child cube, origin xyz=0 0 .1 rpy=0 0 0, axis 0 0 1, limit lower=1 upper=0 effort=0 velocity=vel
- added joint pulley2_axis2: type fixed, parent pulley2, child axis2, origin xyz=0 0 .05 rpy=0 0 0
- added joint tendon2_16_pulley2: type fixed, parent tendon2_16, child pulley2, origin xyz=0 -.55 0 rpy=0 0 0
