Commit message: Firt time a loop is achieved! Still need to fix ho it looks

File: Pendulum_exercise/Inverted_pendulum_tendon_actuation/Cart.urdf (robot description, URDF)
Before this commit: robot myfirst, 1 links, 0 joints
Links:
- link cart: geometry collision box size=0.6 0.1 .3; visual box size=0.6 0.1 .3
