Commit message: Adding two tendons, missing cart

File: Pendulum_exercise/Inverted_pendulum_tendon_actuation/Base_1.urdf (robot description, URDF)
Before this commit: robot myfirst, 1 links, 0 joints
Links:
- added link pulley1, mass 100; collision cylinder length=.1 radius=.5; visual cylinder length=.1 radius=.5
- added link tendon1_1, mass 10; collision cylinder length=.1 radius=.05; visual cylinder length=.1 radius=.05
- added link tendon1_2, mass 10; collision cylinder length=.1 radius=.05; visual cylinder length=.1 radius=.05
- added link tendon1_3, mass 10; collision cylinder length=.1 radius=.05; visual cylinder length=.1 radius=.05
- added link tendon1_4, mass 10; collision cylinder length=.1 radius=.05; visual cylinder length=.1 radius=.05
- added link tendon1_5, mass 10; collision cylinder length=.1 radius=.05; visual cylinder length=.1 radius=.05
Joints:
- added joint Base_pulley1: type revolute, parent Base, child pulley1, origin xyz=.1 .21 .45 rpy=1.57075 0 0, axis 0 0 1, limit lower=1 upper=0 effort=0 velocity=50
- added joint pulley1_tendon1_1: type revolute, parent pulley1, child tendon1_1, origin xyz=0 .55 0 rpy=0 0 0, axis 0 0 1, limit lower=1 upper=0 effort=0 velocity=50
- added joint tendon1_1_tendon1_2: type revolute, parent tendon1_1, child tendon1_2, origin xyz=.4 0 0 rpy=0 0 0, axis 0 0 1, limit lower=1 upper=0 effort=0 velocity=50
- added joint tendon1_2_tendon1_3: type revolute, parent tendon1_2, child tendon1_3, origin xyz=.4 0 0 rpy=0 0 0, axis 0 0 1, limit lower=1 upper=0 effort=0 velocity=50
- added joint tendon1_3_tendon1_4: type revolute, parent tendon1_3, child tendon1_4, origin xyz=.4 0 0 rpy=0 0 0, axis 0 0 1, limit lower=1 upper=0 effort=0 velocity=50
- added joint tendon1_4_tendon1_5: type revolute, parent tendon1_4, child tendon1_5, origin xyz=.4 0 0 rpy=0 0 0, axis 0 0 1, limit lower=1 upper=0 effort=0 velocity=50

Commit message: Cart connetced to tendons and rail

File: Pendulum_exercise/Inverted_pendulum_tendon_actuation/Base_1.urdf (robot description, URDF)
Before this commit: robot myfirst, 7 links, 6 joints
Joints:
- joint Base_pulley1: origin xyz=.1 .21 .45 rpy=1.57075 0 0 -> xyz=.1 .35 .45 rpy=-1.57075 0 0

File: Pendulum_exercise/Inverted_pendulum_tendon_actuation/Rail.urdf (robot description, URDF)
Before this commit: robot myfirst, 1 links, 0 joints
Links:
- added link cart, mass 100; collision box size=0.6 0.3 0.1; visual box size=0.6 0.3 0.1
Joints:
- added joint rail_cart: type prismatic, parent Rail, child cart, origin xyz=0 0 0 rpy=0 1.570796 0, axis 1 0 0, limit lower=-2 upper=2 effort=0 velocity=25

Commit message: Changing bodies configuration

File: Pendulum_exercise/Inverted_pendulum_tendon_actuation/Base_1.urdf (robot description, URDF)
Before this commit: robot myfirst, 7 links, 6 joints
Links:
- removed link tendon1_1
- removed link tendon1_2
- removed link tendon1_3
- removed link tendon1_4
- removed link tendon1_5
Joints:
- removed joint pulley1_tendon1_1
- removed joint tendon1_1_tendon1_2
- removed joint tendon1_2_tendon1_3
- removed joint tendon1_3_tendon1_4
- removed joint tendon1_4_tendon1_5

Commit message: rebuilding tendons, paying attention and writing down frame orientation

File: Pendulum_exercise/Inverted_pendulum_tendon_actuation/Base_1.urdf (robot description, URDF)
Before this commit: robot myfirst, 2 links, 1 joints
Links:
- link Base: geometry collision box size=0.3 0.3 1.5; visual box size=0.3 0.3 1.5
Joints:
- joint Base_pulley1: origin xyz=.1 .35 .45 rpy=-1.57075 0 0 -> xyz=0 .35 .15 rpy=-1.57075 0 0

File: Pendulum_exercise/Inverted_pendulum_tendon_actuation/Rail.urdf (robot description, URDF)
Before this commit: robot myfirst, 2 links, 1 joints
Links:
- added link slider, mass 100; collision box size=0.1 0.6 0.3; visual box size=0.1 0.6 0.3
- added link tendon1_1, mass 10; collision cylinder length=.1 radius=.05; visual cylinder length=.1 radius=.05
- added link tendon1_10, mass 10; collision cylinder length=.1 radius=.05; visual cylinder length=.1 radius=.05
- added link tendon1_11, mass 10; collision cylinder length=.1 radius=.05; visual cylinder length=.1 radius=.05
- added link tendon1_12, mass 10; collision cylinder length=.1 radius=.05; visual cylinder length=.1 radius=.05
- added link tendon1_13, mass 10; collision cylinder length=.1 radius=.05; visual cylinder length=.1 radius=.05
- added link tendon1_14, mass 10; collision cylinder length=.1 radius=.05; visual cylinder length=.1 radius=.05
- added link tendon1_2, mass 10; collision cylinder length=.1 radius=.05; visual cylinder length=.1 radius=.05
- added link tendon1_3, mass 10; collision cylinder length=.1 radius=.05; visual cylinder length=.1 radius=.05
- added link tendon1_4, mass 10; collision cylinder length=.1 radius=.05; visual cylinder length=.1 radius=.05
- added link tendon1_5, mass 10; collision cylinder length=.1 radius=.05; visual cylinder length=.1 radius=.05
- added link tendon1_6, mass 10; collision cylinder length=.1 radius=.05; visual cylinder length=.1 radius=.05
- added link tendon1_7, mass 10; collision cylinder length=.1 radius=.05; visual cylinder length=.1 radius=.05
- added link tendon1_8, mass 10; collision cylinder length=.1 radius=.05; visual cylinder length=.1 radius=.05
- added link tendon1_9, mass 10; collision cylinder length=.1 radius=.05; visual cylinder length=.1 radius=.05
- link cart: geometry collision box size=0.1 0.6 0.3; visual box size=0.1 0.6 0.3
Joints:
- removed joint rail_cart
- added joint cart_tendon1_1: type revolute, parent cart, child tendon1_1, origin xyz=0 .55 0 rpy=0 0 0, axis 0 0 1, limit lower=1 upper=0 effort=0 velocity=50
- added joint rail_slider: type prismatic, parent Rail, child slider, origin xyz=0 0 0 rpy=-1.570796 0 0, axis 0 1 0, limit lower=-2 upper=2 effort=0 velocity=25
- added joint slider_cart: type fixed, parent slider, child cart, origin xyz=0 0 0.3 rpy=0 0 0
- added joint tendon1_10_tendon1_11: type revolute, parent tendon1_10, child tendon1_11, origin xyz=0 .2 0 rpy=0 0 0, axis 0 0 1, limit lower=1 upper=0 effort=0 velocity=50
- added joint tendon1_11_tendon1_12: type revolute, parent tendon1_11, child tendon1_12, origin xyz=0 .2 0 rpy=0 0 0, axis 0 0 1, limit lower=1 upper=0 effort=0 velocity=50
- added joint tendon1_12_tendon1_13: type revolute, parent tendon1_12, child tendon1_13, origin xyz=0 .2 0 rpy=0 0 0, axis 0 0 1, limit lower=1 upper=0 effort=0 velocity=50
- added joint tendon1_13_tendon1_14: type revolute, parent tendon1_13, child tendon1_14, origin xyz=0 .2 0 rpy=0 0 0, axis 0 0 1, limit lower=1 upper=0 effort=0 velocity=50
- added joint tendon1_1_tendon1_2: type revolute, parent tendon1_1, child tendon1_2, origin xyz=0 .2 0 rpy=0 0 0, axis 0 0 1, limit lower=1 upper=0 effort=0 velocity=50
- added joint tendon1_2_tendon1_3: type revolute, parent tendon1_2, child tendon1_3, origin xyz=0 .2 0 rpy=0 0 0, axis 0 0 1, limit lower=1 upper=0 effort=0 velocity=50
- added joint tendon1_3_tendon1_4: type revolute, parent tendon1_3, child tendon1_4, origin xyz=0 .2 0 rpy=0 0 0, axis 0 0 1, limit lower=1 upper=0 effort=0 velocity=50
- added joint tendon1_4_tendon1_5: type revolute, parent tendon1_4, child tendon1_5, origin xyz=0 .2 0 rpy=0 0 0, axis 0 0 1, limit lower=1 upper=0 effort=0 velocity=50
- added joint tendon1_5_tendon1_6: type revolute, parent tendon1_5, child tendon1_6, origin xyz=0 .2 0 rpy=0 0 0, axis 0 0 1, limit lower=1 upper=0 effort=0 velocity=50
- added joint tendon1_6_tendon1_7: type revolute, parent tendon1_6, child tendon1_7, origin xyz=0 .2 0 rpy=0 0 0, axis 0 0 1, limit lower=1 upper=0 effort=0 velocity=50
- added joint tendon1_7_tendon1_8: type revolute, parent tendon1_7, child tendon1_8, origin xyz=0 .2 0 rpy=0 0 0, axis 0 0 1, limit lower=1 upper=0 effort=0 velocity=50
- added joint tendon1_8_tendon1_9: type revolute, parent tendon1_8, child tendon1_9, origin xyz=0 .2 0 rpy=0 0 0, axis 0 0 1, limit lower=1 upper=0 effort=0 velocity=50
- added joint tendon1_9_tendon1_10: type revolute, parent tendon1_9, child tendon1_10, origin xyz=0 .2 0 rpy=0 0 0, axis 0 0 1, limit lower=1 upper=0 effort=0 velocity=50
