Commit message: Building body with simplet urdf files, not using contraints, only 'FixedBase'

File: Pendulum_exercise/Inverted_pendulum_tendon_actuation/Rail.urdf (robot description, URDF)
Before this commit: robot myfirst, 1 links, 0 joints
Links:
- removed link Base
- added link Rail, mass 100; collision cylinder length=3 radius=.05; visual cylinder length=3 radius=.05

Commit message: Building body with simplet urdf files, not using contraints, only 'FixedBase'(2)

File: Pendulum_exercise/Inverted_pendulum_tendon_actuation/Rail.urdf (robot description, URDF)
Before this commit: robot myfirst, 1 links, 0 joints
Links:
- link Rail: geometry collision cylinder length=4 radius=.05; visual cylinder length=4 radius=.05

Commit message: Finishsing second tendon and adding gravity, so far good model behavior observed

File: Pendulum_exercise/Inverted_pendulum_tendon_actuation/Rail.urdf (robot description, URDF)
Before this commit: robot myfirst, 17 links, 16 joints
Links:
- added link tendon2_1, mass 10; collision cylinder length=.1 radius=.05; visual cylinder length=.1 radius=.05
- added link tendon2_10, mass 10; collision cylinder length=.1 radius=.05; visual cylinder length=.1 radius=.05
- added link tendon2_11, mass 10; collision cylinder length=.1 radius=.05; visual cylinder length=.1 radius=.05
- added link tendon2_12, mass 10; collision cylinder length=.1 radius=.05; visual cylinder length=.1 radius=.05
- added link tendon2_13, mass 10; collision cylinder length=.1 radius=.05; visual cylinder length=.1 radius=.05
- added link tendon2_14, mass 10; collision cylinder length=.1 radius=.05; visual cylinder length=.1 radius=.05
- added link tendon2_2, mass 10; collision cylinder length=.1 radius=.05; visual cylinder length=.1 radius=.05
- added link tendon2_3, mass 10; collision cylinder length=.1 radius=.05; visual cylinder length=.1 radius=.05
- added link tendon2_4, mass 10; collision cylinder length=.1 radius=.05; visual cylinder length=.1 radius=.05
- added link tendon2_5, mass 10; collision cylinder length=.1 radius=.05; visual cylinder length=.1 radius=.05
- added link tendon2_6, mass 10; collision cylinder length=.1 radius=.05; visual cylinder length=.1 radius=.05
- added link tendon2_7, mass 10; collision cylinder length=.1 radius=.05; visual cylinder length=.1 radius=.05
- added link tendon2_8, mass 10; collision cylinder length=.1 radius=.05; visual cylinder length=.1 radius=.05
- added link tendon2_9, mass 10; collision cylinder length=.1 radius=.05; visual cylinder length=.1 radius=.05
Joints:
- added joint cart_tendon2_1: type revolute, parent cart, child tendon2_1, origin xyz=0 -.55 0 rpy=0 0 0, axis 0 0 1, limit lower=1 upper=0 effort=0 velocity=50
- added joint tendon2_10_tendon2_11: type revolute, parent tendon2_10, child tendon2_11, origin xyz=0 -.2 0 rpy=0 0 0, axis 0 0 1, limit lower=1 upper=0 effort=0 velocity=50
- added joint tendon2_11_tendon2_12: type revolute, parent tendon2_11, child tendon2_12, origin xyz=0 -.2 0 rpy=0 0 0, axis 0 0 1, limit lower=1 upper=0 effort=0 velocity=50
- added joint tendon2_12_tendon2_13: type revolute, parent tendon2_12, child tendon2_13, origin xyz=0 -.2 0 rpy=0 0 0, axis 0 0 1, limit lower=1 upper=0 effort=0 velocity=50
- added joint tendon2_13_tendon2_14: type revolute, parent tendon2_13, child tendon2_14, origin xyz=0 -.2 0 rpy=0 0 0, axis 0 0 1, limit lower=1 upper=0 effort=0 velocity=50
- added joint tendon2_1_tendon2_2: type revolute, parent tendon2_1, child tendon2_2, origin xyz=0 -.2 0 rpy=0 0 0, axis 0 0 1, limit lower=1 upper=0 effort=0 velocity=50
- added joint tendon2_2_tendon2_3: type revolute, parent tendon2_2, child tendon2_3, origin xyz=0 -.2 0 rpy=0 0 0, axis 0 0 1, limit lower=1 upper=0 effort=0 velocity=50
- added joint tendon2_3_tendon2_4: type revolute, parent tendon2_3, child tendon2_4, origin xyz=0 -.2 0 rpy=0 0 0, axis 0 0 1, limit lower=1 upper=0 effort=0 velocity=50
- added joint tendon2_4_tendon2_5: type revolute, parent tendon2_4, child tendon2_5, origin xyz=0 -.2 0 rpy=0 0 0, axis 0 0 1, limit lower=1 upper=0 effort=0 velocity=50
- added joint tendon2_5_tendon2_6: type revolute, parent tendon2_5, child tendon2_6, origin xyz=0 -.2 0 rpy=0 0 0, axis 0 0 1, limit lower=1 upper=0 effort=0 velocity=50
- added joint tendon2_6_tendon2_7: type revolute, parent tendon2_6, child tendon2_7, origin xyz=0 -.2 0 rpy=0 0 0, axis 0 0 1, limit lower=1 upper=0 effort=0 velocity=50
- added joint tendon2_7_tendon2_8: type revolute, parent tendon2_7, child tendon2_8, origin xyz=0 -.2 0 rpy=0 0 0, axis 0 0 1, limit lower=1 upper=0 effort=0 velocity=50
- added joint tendon2_8_tendon2_9: type revolute, parent tendon2_8, child tendon2_9, origin xyz=0 -.2 0 rpy=0 0 0, axis 0 0 1, limit lower=1 upper=0 effort=0 velocity=50
- added joint tendon2_9_tendon2_10: type revolute, parent tendon2_9, child tendon2_10, origin xyz=0 -.2 0 rpy=0 0 0, axis 0 0 1, limit lower=1 upper=0 effort=0 velocity=50
