Commit message: Working on making the frames or reference coeherent

File: Inverted_pendulum_tendon_actuation/Tendons_Cart_Rail.urdf (robot description, URDF)
Before this commit: robot myfirst, 31 links, 30 joints
Links:
- removed link tendon2_1
- removed link tendon2_10
- removed link tendon2_11
- removed link tendon2_12
- removed link tendon2_13
- removed link tendon2_14
- removed link tendon2_2
- removed link tendon2_3
- removed link tendon2_4
- removed link tendon2_5
- removed link tendon2_6
- removed link tendon2_7
- removed link tendon2_8
- removed link tendon2_9
Joints:
- removed joint cart_tendon2_1
- removed joint tendon2_10_tendon2_11
- removed joint tendon2_11_tendon2_12
- removed joint tendon2_12_tendon2_13
- removed joint tendon2_13_tendon2_14
- removed joint tendon2_1_tendon2_2
- removed joint tendon2_2_tendon2_3
- removed joint tendon2_3_tendon2_4
- removed joint tendon2_4_tendon2_5
- removed joint tendon2_5_tendon2_6
- removed joint tendon2_6_tendon2_7
- removed joint tendon2_7_tendon2_8
- removed joint tendon2_8_tendon2_9
- removed joint tendon2_9_tendon2_10
