Commit message: Adding a pendulum and setting motors to a initial state off to avoid unwanted friction

File: Inverted_pendulum_tendon_actuation/Tendon_1_Cart_Rail.urdf (robot description, URDF)
Before this commit: robot myfirst, 17 links, 16 joints
Links:
- added link pendulum, mass 100; collision box size=0.1 0.8 .1; visual box size=0.1 0.8 .1
- added link pendulumAxis, mass 100; collision box size=0.1 0.1 .1; visual box size=0.1 0.1 .1
Joints:
- added joint cart_pendulumAxis: type revolute, parent cart, child pendulumAxis, origin xyz=0 0 .21 rpy=0 0 0, axis 0 0 1, limit lower=1 upper=0 effort=0 velocity=205
- added joint pendulumAxis_pendulum: type fixed, parent pendulumAxis, child pendulum, origin xyz=-0.45 0 0 rpy=0 0 1.570796
