Commit message: Reference point:tendon_pendulum_balanced_Little_external_hep, pulleys masses were reduced by 10, pendulum lenght was doubled

File: Inverted_pendulum_tendon_actuation/Base_1.urdf (robot description, URDF)
Before this commit: robot myfirst, 2 links, 1 joints
Links:
- link pulley1: mass 100 -> 2

File: Inverted_pendulum_tendon_actuation/Base_2.urdf (robot description, URDF)
Before this commit: robot myfirst, 16 links, 15 joints
Links:
- link pulley1: mass 100 -> 2

File: Inverted_pendulum_tendon_actuation/Pendulum_Tendon_1_Cart_Rail.urdf (robot description, URDF)
Before this commit: robot myfirst, 19 links, 18 joints
Links:
- link pendulum: mass 100 -> 1; geometry collision box size=0.1 2 .1; visual box size=0.1 2 .1
- link pendulumAxis: mass 100 -> 10
Joints:
- joint cart_pendulumAxis: origin xyz=0 0 .21 rpy=0 0 3.1416 -> xyz=0 0 .21 rpy=0 0 0
- joint pendulumAxis_pendulum: origin xyz=-0.45 0 0 rpy=0 0 1.570796 -> xyz=1 0 0 rpy=0 0 1.570796
